File: hardware/pcb/frameprobe.kicad_sch (KiCad schematic)
At the start: 18 parts, among them U1 TLV9061IDBVR, U2 RP2040-Zero

Commit message: rename to frameprobe
Parts:
- D1: footprint click2photon:VBPW34S -> frameprobe:VBPW34S; symbol click2photon:VBPW34S -> frameprobe:VBPW34S
- U2: footprint click2photon:RP2040-Zero_THT -> frameprobe:RP2040-Zero_THT; symbol click2photon:RP2040-Zero -> frameprobe:RP2040-Zero
Other:
- note added: "frameprobe — display-latency sensor TLV9061 TIA + BPW34S photodiode + RP2040-Zero carrier"
- note removed: "click2photon — display-latency sensor TLV9061 TIA + BPW34S photodiode + RP2040-Zero carrier"
Changed lines of the file:
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@@
 		)
 	)
-	(text "click2photon — display-latency sensor\nTLV9061 TIA + BPW34S photodiode + RP2040-Zero carrier"
+	(text "frameprobe — display-latency sensor\nTLV9061 TIA + BPW34S photodiode + RP2040-Zero carrier"
 		(exclude_from_sim no)
 		(at 99.06 45.72 0)
@@
 		)
 		(instances
-			(project "click2photon"
+			(project "frameprobe"
 				(path "/e5f9a1c0-0000-4000-8000-c11c42070001"
 					(reference "U1")
@@
 	)
 	(symbol
-		(lib_id "click2photon:RP2040-Zero")
+		(lib_id "frameprobe:RP2040-Zero")
 		(at 215.9 96.52 0)
 		(unit 1)
@@
 			)
 		)
-		(property "Footprint" "click2photon:RP2040-Zero_THT"
+		(property "Footprint" "frameprobe:RP2040-Zero_THT"
 			(at 215.9 96.52 0)
 			(show_name no)
@@
 		)
 		(instances
-			(project "click2photon"
+			(project "frameprobe"
 				(path "/e5f9a1c0-0000-4000-8000-c11c42070001"
 					(reference "U2")
@@
 	)
 	(symbol
-		(lib_id "click2photon:VBPW34S")
+		(lib_id "frameprobe:VBPW34S")
 		(at 118.11 101.6 180)
 		(unit 1)
@@
 			)
 		)
-		(property "Footprint" "click2photon:VBPW34S"
+		(property "Footprint" "frameprobe:VBPW34S"
 			(at 118.11 101.6 0)
 			(show_name no)
@@
 		)
 		(instances
-			(project "click2photon"
+			(project "frameprobe"
 				(path "/e5f9a1c0-0000-4000-8000-c11c42070001"
 					(reference "D1")
@@
 		)
 		(instances
-			(project "click2photon"
+			(project "frameprobe"
 				(path "/e5f9a1c0-0000-4000-8000-c11c42070001"
 					(reference "R1")
@@
 		)
 		(instances
-			(project "click2photon"
+			(project "frameprobe"
 				(path "/e5f9a1c0-0000-4000-8000-c11c42070001"
 					(reference "R2")
@@
 		)
 		(instances
-			(project "click2photon"
+			(project "frameprobe"
 				(path "/e5f9a1c0-0000-4000-8000-c11c42070001"
 					(reference "R3")
@@
 		)
 		(instances
-			(project "click2photon"
+			(project "frameprobe"
 				(path "/e5f9a1c0-0000-4000-8000-c11c42070001"
 					(reference "R4")
@@
 		)
 		(instances
-			(project "click2photon"
+			(project "frameprobe"
 				(path "/e5f9a1c0-0000-4000-8000-c11c42070001"
 					(reference "C1")
@@
 		)
 		(instances
-			(project "click2photon"
+			(project "frameprobe"
 				(path "/e5f9a1c0-0000-4000-8000-c11c42070001"
 					(reference "C2")
@@
 		)
 		(instances
-			(project "click2photon"
+			(project "frameprobe"
 				(path "/e5f9a1c0-0000-4000-8000-c11c42070001"
 					(reference "C3")
@@
 		)
 		(instances
-			(project "click2photon"
+			(project "frameprobe"
 				(path "/e5f9a1c0-0000-4000-8000-c11c42070001"
 					(reference "C4")
@@
 		)
 		(instances
-			(project "click2photon"
+			(project "frameprobe"
 				(path "/e5f9a1c0-0000-4000-8000-c11c42070001"
 					(reference "C5")
@@
 		)
 		(instances
-			(project "click2photon"
+			(project "frameprobe"
 				(path "/e5f9a1c0-0000-4000-8000-c11c42070001"
 					(reference "TP1")
@@
 		)
 		(instances
-			(project "click2photon"
+			(project "frameprobe"
 				(path "/e5f9a1c0-0000-4000-8000-c11c42070001"
 					(reference "TP2")
@@
 		)
 		(instances
-			(project "click2photon"
+			(project "frameprobe"
 				(path "/e5f9a1c0-0000-4000-8000-c11c42070001"
 					(reference "H1")
@@
 		)
 		(instances
-			(project "click2photon"
+			(project "frameprobe"
 				(path "/e5f9a1c0-0000-4000-8000-c11c42070001"
 					(reference "H2")
@@
 		)
 		(instances
-			(project "click2photon"
+			(project "frameprobe"
 				(path "/e5f9a1c0-0000-4000-8000-c11c42070001"
 					(reference "H3")
@@
 		)
 		(instances
-			(project "click2photon"
+			(project "frameprobe"
 				(path "/e5f9a1c0-0000-4000-8000-c11c42070001"
 					(reference "H4")
@@
 		)
 		(instances
-			(project "click2photon"
+			(project "frameprobe"
 				(path "/e5f9a1c0-0000-4000-8000-c11c42070001"
 					(reference "#PWR01")
@@
 		)
 		(instances
-			(project "click2photon"
+			(project "frameprobe"
 				(path "/e5f9a1c0-0000-4000-8000-c11c42070001"
 					(reference "#PWR02")
@@
 		)
 		(instances
-			(project "click2photon"
+			(project "frameprobe"
 				(path "/e5f9a1c0-0000-4000-8000-c11c42070001"
 					(reference "#PWR03")
@@
 		)
 		(instances
-			(project "click2photon"
+			(project "frameprobe"
 				(path "/e5f9a1c0-0000-4000-8000-c11c42070001"
 					(reference "#PWR04")
@@
 		)
 		(instances
-			(project "click2photon"
+			(project "frameprobe"
 				(path "/e5f9a1c0-0000-4000-8000-c11c42070001"
 					(reference "#PWR05")
@@
 		)
 		(instances
-			(project "click2photon"
+			(project "frameprobe"
 				(path "/e5f9a1c0-0000-4000-8000-c11c42070001"
 					(reference "#PWR06")
@@
 		)
 		(instances
-			(project "click2photon"
+			(project "frameprobe"
 				(path "/e5f9a1c0-0000-4000-8000-c11c42070001"
 					(reference "#PWR07")
@@
 		)
 		(instances
-			(project "click2photon"
+			(project "frameprobe"
 				(path "/e5f9a1c0-0000-4000-8000-c11c42070001"
 					(reference "#PWR08")
@@
 		)
 		(instances
-			(project "click2photon"
+			(project "frameprobe"
 				(path "/e5f9a1c0-0000-4000-8000-c11c42070001"
 					(reference "#PWR09")
@@
 		)
 		(instances
-			(project "click2photon"
+			(project "frameprobe"
 				(path "/e5f9a1c0-0000-4000-8000-c11c42070001"
 					(reference "#PWR10")
@@
 		)
 		(instances
-			(project "click2photon"
+			(project "frameprobe"
 				(path "/e5f9a1c0-0000-4000-8000-c11c42070001"
 					(reference "#PWR11")
@@
 		)
 		(instances
-			(project "click2photon"
+			(project "frameprobe"
 				(path "/e5f9a1c0-0000-4000-8000-c11c42070001"
 					(reference "#PWR12")
@@
 		)
 		(instances
-			(project "click2photon"
+			(project "frameprobe"
 				(path "/e5f9a1c0-0000-4000-8000-c11c42070001"
 					(reference "#PWR13")
@@
 		)
 		(instances
-			(project "click2photon"
+			(project "frameprobe"
 				(path "/e5f9a1c0-0000-4000-8000-c11c42070001"
 					(reference "#PWR14")
