File: hardware/pcb/frameprobe.kicad_pcb (KiCad board)
At the start: 2 copper layers, 30 x 48 mm, 18 parts, among them U1 TLV9061IDBVR, U2 RP2040-Zero

Commit message: rename to frameprobe
Parts:
- D1: footprint click2photon:VBPW34S -> frameprobe:VBPW34S
- U2: footprint click2photon:RP2040-Zero_THT -> frameprobe:RP2040-Zero_THT
Other:
- board text added: "frameprobe"
- board text added: "frameprobe rev2"
- board text removed: "click2photon"
- board text removed: "click2photon rev2"
Changed lines of the file:
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@@
 		)
 	)
-	(footprint "click2photon:VBPW34S"
+	(footprint "frameprobe:VBPW34S"
 		(layer "F.Cu")
 		(at 111.5 129.5 180)
@@
 		(embedded_fonts no)
 	)
-	(footprint "click2photon:RP2040-Zero_THT"
+	(footprint "frameprobe:RP2040-Zero_THT"
 		(layer "B.Cu")
 		(at 115 111.75 180)
@@
 		)
 	)
-	(gr_text "click2photon rev2"
+	(gr_text "frameprobe rev2"
 		(at 128 133 90)
 		(layer "F.SilkS")
@@
 		)
 	)
-	(gr_text "click2photon"
+	(gr_text "frameprobe"
 		(at 124 138 0)
 		(layer "B.SilkS")

Commit message: pcb text
Other:
- board text added: "frameprobe rev2 batch no. 1"
- board text added: "info@frameprobe.com"
- board text removed: "frameprobe"
Changed lines of the file:
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@@
 		)
 	)
-	(gr_text "frameprobe rev2"
-		(at 128 133 90)
+	(gr_text "frameprobe rev2\nbatch no. 1"
+		(at 127.85 133 90)
 		(layer "F.SilkS")
 		(effects
@@
 		)
 	)
-	(gr_text "frameprobe"
-		(at 124 138 0)
+	(gr_text "info@frameprobe.com"
+		(at 115 143.4 0)
 		(layer "B.SilkS")
 		(effects
+			(font
+				(size 1 1)
+				(thickness 0.15)
+			)
+			(justify mirror)
+		)
+	)
+	(gr_text "frameprobe rev2"
+		(at 122.5 138 0)
+		(layer "B.SilkS")
+		(effects
